File: cad/HabitatCAN Dev Board (ESP32).kicad_pcb (KiCad board)
At the start: 2 copper layers, 85.5 x 48 mm, 68 parts, among them J1 GPIO Connection, J2 CAN Data, J3 CAN Data (HabitatCAN Interfac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, J4 24v Bus Power, J5 USB_C_Receptacle_USB2.0, SW1 Reset, SW2 Boot, U1 ESP32-C3-MINI-1, U2 AMS1117-3.3, U3 TJA1051T, U4 OKI-78SR

Commit message: Updated to Rev4
Parts:
- added C12: 10uF / 25v (20%), Capacitor_SMD:C_0603_1608Metric, F.Cu at (96.9, 101.3)
- added G***: LOGO, Qwiic:qwiic_7mm, F.Cu at (99.7, 95.2)
- added J6: Qwiic Connector, Connector_JST:JST_SH_BM04B-SRSS-TB_1x04-1MP_P1.00mm_Vertical, F.Cu at (95.3, 95.4)
- moved REF** 73.6 mm to (164.5, 124.2), turned to 0 degrees
Routing:
- net +3V3: track 86.3 -> 110.3 mm, vias 2 -> 4
- net GPIO7: track 43.6 -> 67.4 mm, vias 0 -> 2
- net GPIO6: track 40.8 -> 64.5 mm, vias 0 -> 2
- net GPIO4: track 94.1 -> 97.5 mm
- net GPIO5: track 88.8 -> 92.0 mm
Other:
- board text added: "Rev 4 25/09/15"
- board text removed: "Rev 3 25/09/14"
