File: cad/HabitatCAN Dev Board (ESP32).kicad_sch (KiCad schematic)
At the start: 20 parts, among them J1 GPIO Connection, J2 CAN Data, J3 CAN Data (HabitatCAN Interfac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, J4 24v Bus Power, SW1 Reset, SW2 Boot, U4 OKI-78SR

Commit message: Updated to Rev4
Parts:
- added C12: 10uF / 25v (20%), Capacitor_SMD:C_0603_1608Metric, symbol Device:C
- added J6: Qwiic Connector, Connector_JST:JST_SH_BM04B-SRSS-TB_1x04-1MP_P1.00mm_Vertical, symbol Connector_Generic:Conn_01x04
Connections:
- net +3V3: now also C12.2, J6.2 (Pin_2)
- net GND: now also C12.1, J6.1 (Pin_1)
- net GPIO6: now also J6.3 (Pin_3)
- net GPIO7: now also J6.4 (Pin_4)
Other:
- moved on the sheet: H1, H2, H3, H4
